File: pcb/hhkb_400.kicad_pcb (KiCad board)
At the start: 2 copper layers, 285.8 x 101.2 mm, 158 parts, among them J1 USB_mini_micro_B, SW1 SW_PUSH, U1 ATMEGA32U4, X1 XTAL_GND

Commit message: use jumper to represent jumper, rather than 0ohm resister
Parts:
- removed JMP1:6, JMP1:7, JMP3, JMP4, JMP4:4: 0, Resistors_SMD:R_1206_HandSoldering
- removed JP2:0: Jumper, Resistors_SMD:R_1206_HandSoldering
- removed Poker_oval_hole (x6): VAL**, keyboard_parts:Poker_oval_hole
- added JP_C4: Jumper, Resistors_SMD:R_1206_HandSoldering, B.Cu at (105.4, 83.3)
- added JP_C6: Jumper, Resistors_SMD:R_1206_HandSoldering, B.Cu at (135.8, 82.5)
- added JP_C7: Jumper, Resistors_SMD:R_1206_HandSoldering, B.Cu at (147.5, 85.5)
- added JP_R2: Jumper, Resistors_SMD:R_1206_HandSoldering, B.Cu at (166.1, 85.4)
- added JP_R3: Jumper, Resistors_SMD:R_1206_HandSoldering, B.Cu at (128.5, 76.0)
- added JP_R4: Jumper, Resistors_SMD:R_1206_HandSoldering, B.Cu at (131.2, 76.0)
Routing:
- net GND: track 686.2 -> 689.3 mm
- net /COL6: track 8.13 -> 5.52 mm
- net /COL7: track 20.5 -> 19.9 mm

Commit message: update
Parts:
- moved ","1 97.2 mm to (253.6, 158.1)
- moved "."1 97.2 mm to (272.7, 158.1)
- moved "B"1 97.2 mm to (196.5, 158.1)
- moved "C"1 97.2 mm to (158.4, 158.1)
- moved "M"1 97.2 mm to (234.6, 158.1)
- moved "N"1 97.2 mm to (215.5, 158.1)
- moved "V"1 97.2 mm to (177.4, 158.1)
- moved "X"1 97.2 mm to (139.3, 158.1)
- moved "Z"1 97.2 mm to (120.3, 158.1)
- moved "["1 97.2 mm to (296.5, 120.0)
- moved D1:11 97.2 mm to (281.3, 104.5)
- moved D2:10 97.2 mm to (265.6, 123.6)
- moved D3:11 97.2 mm to (286.1, 142.6)
- moved D5:4 97.2 mm to (226.4, 168.6)
- moved JP_C3 97.2 mm to (150.4, 162.8)
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Routing:
- net VCC: track 303.0 -> 303.7 mm
