File: pcb/hhkb.sch (KiCad schematic (older format))
At the start: 150 parts, among them J1 USB_mini_micro_B, SW1 SW_PUSH, U1 ATMEGA32U4, X1 XTAL_GND

Commit message: enlarge trace width
Parts:
- removed JP9, JP_C10, JP_C3, JP_C4, JP_C5, JP_C6, JP_C7, JP_C8, JP_C9re1, JP_GND1, JP_GND2, JP_R2, JP_R3, JP_R4: Jumper, Resistors_SMD:R_1206_HandSoldering, symbol Jumper
- SPACEBAR1: footprint TheKeebrary:MX_Plate_400H -> TheKeebrary:MX_Plate_600H_Stepped
- U1: symbol ATmega32U4 -> ATMEGA32U4
- renumbered D4:9 to D10:10, D5:5 to D10:11, D5:6 to D10:12, D3:8 to D10:7, D4:7 to D10:8, D4:8 to D10:9, D1:7 to D2:6, D2:6 to D3:6, D4:2 to D4:1, D4:3 to D4:2, D4:4 to D4:3, D4:5 to D4:4, D3:6 to D4:5, D2:7 to D4:6, D4:1 to D5:1, D5:1 to D5:2, D5:2 to D5:3, D4:6 to D5:4, D3:7 to D5:5, D5:4 to D5:6, D1:15 to D6:12, D1:10 to D6:7, D1:11 to D6:8, D1:12 to D6:9, D2:12 to D7:10, D2:13 to D7:11, D2:14 to D7:12, D2:10 to D7:8, D2:11 to D7:9, D3:11 to D8:10, D3:12 to D8:11, D3:13 to D8:12, D1:8 to D8:7, D2:9 to D8:8, D3:10 to D8:9, D4:11 to D9:10, D4:12 to D9:11, D4:13 to D9:12, D2:8 to D9:7, D3:9 to D9:8, D4:10 to D9:9, D1:13 to D:6:10, D1:14 to D:6:11, D1:9 to D:7:7
Connections:
- net labels added: D+, D-, ROW10, ROW6, ROW7, ROW8, ROW9
- net labels removed: COL13, COL14, COL15
- wire segments 200 -> 197
- no-connect marks 7 -> 5
Other:
- moved on the sheet: "'"1, ","1, "-"1, "."1, "/"1, "0"1, "1"1, "2"1, "3"1, "4"1, "5"1, "6"1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

Commit message: fix left super size
Parts:
- L_CMD1: footprint TheKeebrary:MX_Plate_100H -> TheKeebrary:MX_Plate_150H
Changed lines of the file:
@@
 F 0 "L_CMD1" H 3550 6150 60  0000 C CNN
 F 1 "KEYSW" H 3600 6050 60  0001 C CNN
-F 2 "TheKeebrary:MX_Plate_100H" H 3600 6150 60  0001 C CNN
+F 2 "TheKeebrary:MX_Plate_150H" H 3600 6150 60  0001 C CNN
 F 3 "" H 3600 6150 60  0000 C CNN
 	1    3600 6150
