File: pcb/hhkb.kicad_pcb (KiCad board)
At the start: 2 copper layers, 285.8 x 100.6 mm, 150 parts, among them J1 USB_mini_micro_B, SW1 SW_PUSH, U1 ATMEGA32U4, X1 XTAL_GND

Commit message: rework pcb artwork
Parts:
- removed D1:10, D1:11, D1:12, D1:13, D1:14, D1:15, D1:7, D1:8, D1:9, D2:10, D2:11, D2:12, D2:13, D2:14, D2:7, D2:8, D2:9, D3:10, D3:11, D3:12, D3:13, D3:7, D3:8, D3:9, D4:10, D4:11, D4:12, D4:13, D4:7, D4:8, D4:9: D, Diodes_SMD:D_SOD-123
- removed JP9, JP_C10, JP_C3, JP_C4, JP_C5, JP_C6, JP_C7, JP_C8, JP_C9re1, JP_GND1, JP_GND2, JP_R2, JP_R3, JP_R4: Jumper, Resistors_SMD:R_1206_HandSoldering
- added D10:10: D, Diodes_SMD:D_SOD-123, B.Cu at (245.6, 157.3)
- added D10:11: D, Diodes_SMD:D_SOD-123, B.Cu at (252.3, 162.7)
- added D10:12: D, Diodes_SMD:D_SOD-123, B.Cu at (255.2, 162.7)
- added D10:7: D, Diodes_SMD:D_SOD-123, B.Cu at (214.2, 148.1)
- added D10:8: D, Diodes_SMD:D_SOD-123, B.Cu at (214.2, 150.3)
- added D10:9: D, Diodes_SMD:D_SOD-123, B.Cu at (228.0, 153.7)
- added D5:3: D, Diodes_SMD:D_SOD-123, B.Cu at (127.4, 176.7)
- added D6:12: D, Diodes_SMD:D_SOD-123, B.Cu at (348.0, 97.7)
- added D6:7: D, Diodes_SMD:D_SOD-123, B.Cu at (254.2, 97.7)
- added D6:8: D, Diodes_SMD:D_SOD-123, B.Cu at (271.6, 97.7)
- added D6:9: D, Diodes_SMD:D_SOD-123, B.Cu at (293.8, 97.7)
- added D7:10: D, Diodes_SMD:D_SOD-123, B.Cu at (300.6, 98.7)
- added D7:11: D, Diodes_SMD:D_SOD-123, B.Cu at (319.2, 98.7)
- added D7:12: D, Diodes_SMD:D_SOD-123, B.Cu at (335.8, 98.7)
- added D7:8: D, Diodes_SMD:D_SOD-123, B.Cu at (275.7, 98.7)
- added D7:9: D, Diodes_SMD:D_SOD-123, B.Cu at (282.6, 98.7)
- added D8:10: D, Diodes_SMD:D_SOD-123, B.Cu at (296.6, 99.7)
- added D8:11: D, Diodes_SMD:D_SOD-123, B.Cu at (315.6, 99.7)
- added D8:12: D, Diodes_SMD:D_SOD-123, B.Cu at (331.8, 99.7)
- added D8:7: D, Diodes_SMD:D_SOD-123, B.Cu at (220.6, 99.7)
- added D8:8: D, Diodes_SMD:D_SOD-123, B.Cu at (259.4, 99.7)
- added D8:9: D, Diodes_SMD:D_SOD-123, B.Cu at (279.2, 99.7)
- added D9:10: D, Diodes_SMD:D_SOD-123, B.Cu at (274.2, 165.7)
- added D9:11: D, Diodes_SMD:D_SOD-123, B.Cu at (278.6, 165.3)
- added D9:12: D, Diodes_SMD:D_SOD-123, B.Cu at (278.6, 167.3)
- added D9:7: D, Diodes_SMD:D_SOD-123, B.Cu at (235.2, 149.5)
- added D9:8: D, Diodes_SMD:D_SOD-123, B.Cu at (239.6, 149.5)
- added D9:9: D, Diodes_SMD:D_SOD-123, B.Cu at (272.6, 165.7)
- added D:6:10: D, Diodes_SMD:D_SOD-123, B.Cu at (312.0, 97.7)
- added D:6:11: D, Diodes_SMD:D_SOD-123, B.Cu at (329.0, 97.7)
- added D:7:7: D, Diodes_SMD:D_SOD-123, B.Cu at (239.8, 98.7)
- SPACEBAR1: footprint TheKeebrary:MX_Plate_400H -> TheKeebrary:MX_Plate_600H_Stepped
- moved J1 209.5 mm to (315.6, 91.4)
- moved D5:6 81.1 mm to (203.4, 177.6), turned to 0 degrees
- moved D5:5 76.4 mm to (201.8, 171.7), turned to 90 degrees
- moved C6 70.2 mm to (236.2, 181.9), turned to 225 degrees
- moved C8 67.7 mm to (240.0, 180.9), turned to 315 degrees
- moved C7 64.1 mm to (246.3, 176.7)
- moved R1 60.2 mm to (230.6, 176.9)
- moved C3 58.9 mm to (246.3, 178.7)
- moved U1 55.2 mm to (239.2, 171.0), turned to 90 degrees
- moved C1 55.0 mm to (225.6, 173.9), turned to 135 degrees
- moved X1 54.4 mm to (227.9, 171.7), turned to 135 degrees
- moved SW1 51.8 mm to (218.2, 166.6), turned to 270 degrees
- moved C4 49.6 mm to (246.3, 165.2)
- moved R2 49.6 mm to (246.3, 163.0)
- moved C2 47.6 mm to (224.4, 170.3), turned to 225 degrees
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Connections:
- "'"1 pad 1: Net-("'"1-Pad1) -> /COL11
- "'"1 pad 2: /COL14 -> Net-("'"1-Pad2)
- ","1 pad 1: Net-(","1-Pad1) -> /COL10
- ","1 pad 2: /COL12 -> Net-(","1-Pad2)
- "-"1 pad 1: Net-("-"1-Pad1) -> /COL9
- "-"1 pad 2: /COL12 -> Net-("-"1-Pad2)
- "."1 pad 1: Net-("."1-Pad1) -> /COL9
- "."1 pad 2: /COL13 -> Net-("."1-Pad2)
- "/"1 pad 1: Net-("/"1-Pad1) -> /COL10
- "/"1 pad 2: /COL14 -> Net-("/"1-Pad2)
- "0"1 pad 1: Net-("0"1-Pad1) -> /COL8
- "0"1 pad 2: /COL11 -> Net-("0"1-Pad2)
- "2"1 pad 1: Net-("2"1-Pad1) -> /COL3
- "3"1 pad 1: Net-("3"1-Pad1) -> /COL4
- "4"1 pad 1: Net-("4"1-Pad1) -> /COL5
- "5"1 pad 1: Net-("5"1-Pad1) -> /COL6
- "6"1 pad 1: Net-("6"1-Pad1) -> /COL6
- "7"1 pad 1: Net-("7"1-Pad1) -> /COL7
- "8"1 pad 1: Net-("8"1-Pad1) -> /COL7
- "9"1 pad 1: Net-("9"1-Pad1) -> /COL7
- ";"1 pad 1: Net-(";"1-Pad1) -> /COL10
- ";"1 pad 2: /COL13 -> Net-(";"1-Pad2)
- "="1 pad 1: Net-("="1-Pad1) -> /COL10
- "="1 pad 2: /COL13 -> Net-("="1-Pad2)
- "B"1 pad 1: Net-("B"1-Pad1) -> /COL4
- "C"1 pad 1: Net-("3"1-Pad1) -> /COL3
- "D"1 pad 1: Net-("3"1-Pad1) -> /COL4
- "E"1 pad 1: Net-("3"1-Pad1) -> /COL4
- "F"1 pad 1: Net-("4"1-Pad1) -> /COL5
- "G"1 pad 1: Net-("7"1-Pad1) -> /COL5
- "H"1 pad 1: Net-("8"1-Pad1) -> /COL5
- "I"1 pad 1: Net-("9"1-Pad1) -> /COL8
- "J"1 pad 1: Net-("9"1-Pad1) -> /COL7
- "K"1 pad 1: Net-("K"1-Pad1) -> /COL8
- "K"1 pad 2: /COL11 -> Net-("K"1-Pad2)
- "L"1 pad 1: Net-("L"1-Pad1) -> /COL9
- "L"1 pad 2: /COL12 -> Net-("L"1-Pad2)
- "M"1 pad 1: Net-("M"1-Pad1) -> /COL9
- "M"1 pad 2: /COL11 -> Net-("M"1-Pad2)
- "N"1 pad 1: Net-("9"1-Pad1) -> /COL8
- "O"1 pad 1: Net-("O"1-Pad1) -> /COL8
- "O"1 pad 2: /COL11 -> Net-("O"1-Pad2)
- "P"1 pad 1: Net-("P"1-Pad1) -> /COL9
- "P"1 pad 2: /COL12 -> Net-("P"1-Pad2)
- "R"1 pad 1: Net-("4"1-Pad1) -> /COL5
- "S"1 pad 1: Net-("2"1-Pad1) -> /COL3
- "T"1 pad 1: Net-("6"1-Pad1) -> /COL6
- "U"1 pad 1: Net-("8"1-Pad1) -> /COL7
- "V"1 pad 1: Net-("6"1-Pad1) -> /COL4
- "W"1 pad 1: Net-("2"1-Pad1) -> /COL3
- "X"1 pad 1: Net-("2"1-Pad1) -> /COL2
- "Y"1 pad 1: Net-("7"1-Pad1) -> /COL6
- "Z"1 pad 1: /COL2 -> /COL1
- "["1 pad 1: Net-("["1-Pad1) -> /COL10
- "["1 pad 2: /COL13 -> Net-("["1-Pad2)
- "\"1 pad 1: Net-("\"1-Pad1) -> /COL11
- "\"1 pad 2: /COL14 -> Net-("\"1-Pad2)
- "]"1 pad 1: Net-("]"1-Pad1) -> /COL11
- "]"1 pad 2: /COL14 -> Net-("]"1-Pad2)
- "`"1 pad 1: Net-("`"1-Pad1) -> /COL12
- "`"1 pad 2: /COL15 -> Net-("`"1-Pad2)
- ALT1 pad 1: /COL1 -> /COL2
- BS1 pad 1: Net-(BS1-Pad1) -> /COL12
- BS1 pad 2: /COL15 -> Net-(BS1-Pad2)
- D2:1 pad 1: Net-(D2:1-Pad1) -> /ROW2
- D2:2 pad 1: Net-(D2:1-Pad1) -> /ROW2
- D2:3 pad 1: Net-(D2:1-Pad1) -> /ROW2
- D2:4 pad 1: Net-(D2:1-Pad1) -> /ROW2
- D2:5 pad 1: Net-(D2:1-Pad1) -> /ROW2
- D2:6 pad 1: Net-(D2:1-Pad1) -> /ROW2
- D2:6 pad 2: Net-("T"1-Pad2) -> Net-("6"1-Pad2)
- D3:1 pad 1: Net-(D3:1-Pad1) -> /ROW3
- D3:2 pad 1: Net-(D3:1-Pad1) -> /ROW3
- D3:3 pad 1: Net-(D3:1-Pad1) -> /ROW3
- D3:4 pad 1: Net-(D3:1-Pad1) -> /ROW3
- D3:5 pad 1: Net-(D3:1-Pad1) -> /ROW3
- D3:6 pad 1: Net-(D3:1-Pad1) -> /ROW3
- D3:6 pad 2: Net-("G"1-Pad2) -> Net-("T"1-Pad2)
- D4:1 pad 1: Net-(D4:1-Pad1) -> /ROW4
- D4:1 pad 2: Net-(D4:1-Pad2) -> Net-("Z"1-Pad2)
- D4:2 pad 1: Net-(D4:1-Pad1) -> /ROW4
- D4:2 pad 2: Net-("Z"1-Pad2) -> Net-("X"1-Pad2)
- D4:3 pad 1: Net-(D4:1-Pad1) -> /ROW4
- D4:3 pad 2: Net-("X"1-Pad2) -> Net-("C"1-Pad2)
- D4:4 pad 1: Net-(D4:1-Pad1) -> /ROW4
- D4:4 pad 2: Net-("C"1-Pad2) -> Net-("V"1-Pad2)
- D4:5 pad 1: Net-(D3:1-Pad1) -> /ROW4
- D4:5 pad 2: Net-("V"1-Pad2) -> Net-("G"1-Pad2)
- D4:6 pad 1: Net-(D4:1-Pad1) -> /ROW4
- D4:6 pad 2: Net-("B"1-Pad2) -> Net-("Y"1-Pad2)
- D5:1 pad 2: Net-(ALT1-Pad2) -> Net-(D5:1-Pad2)
- D5:2 pad 2: Net-(D5:2-Pad2) -> Net-(ALT1-Pad2)
- D5:4 pad 2: Net-(D5:4-Pad2) -> Net-("B"1-Pad2)
- D5:5 pad 2: Net-(D5:5-Pad2) -> Net-("H"1-Pad2)
- L_CMD1 pad 1: /COL2 -> /COL3
- L_CMD1 pad 2: Net-(D5:2-Pad2) -> Net-(D5:3-Pad2)
- L_SHIFT1 pad 2: Net-(D4:1-Pad2) -> Net-(D5:1-Pad2)
- RET1 pad 1: Net-(D3:13-Pad2) -> /COL12
- RET1 pad 2: /COL15 -> Net-(D8:12-Pad2)
- R_ALT1 pad 1: Net-(D5:6-Pad2) -> /COL12
- R_ALT1 pad 2: /COL14 -> Net-(D10:12-Pad2)
- R_CMD1 pad 1: Net-(D5:5-Pad2) -> /COL11
- R_CMD1 pad 2: /COL13 -> Net-(D10:11-Pad2)
- R_FN1 pad 1: Net-(D4:13-Pad2) -> /COL12
- R_FN1 pad 2: /COL15 -> Net-(D9:12-Pad2)
- R_SHIFT1 pad 1: Net-(D4:12-Pad2) -> /COL11
- R_SHIFT1 pad 2: /COL15 -> Net-(D9:11-Pad2)
- SPACEBAR1 pad 1: /COL10 -> /COL6
- SPACEBAR1 pad 2: Net-(D5:4-Pad2) -> Net-(D5:6-Pad2)
- U1 pad 12: /COL4 -> /ROW4
- U1 pad 18: /ROW3 -> Net-(U1-Pad18)
- U1 pad 19: /ROW4 -> Net-(U1-Pad19)
- U1 pad 20: /COL5 -> /COL4
- U1 pad 21: Net-(U1-Pad21) -> /COL5
- U1 pad 22: Net-(U1-Pad22) -> /COL6
- U1 pad 25: /COL6 -> /ROW3
- U1 pad 26: /COL7 -> /ROW2
- U1 pad 27: Net-(U1-Pad27) -> /ROW1
- U1 pad 28: Net-(U1-Pad28) -> /COL7
- U1 pad 30: /COL9 -> /ROW10
- U1 pad 31: /COL10 -> /COL9
- U1 pad 32: /ROW2 -> /ROW9
- U1 pad 36: /COL11 -> /COL10
- U1 pad 37: /COL12 -> /COL11
- U1 pad 38: /COL13 -> /COL12
- U1 pad 39: /COL14 -> /ROW8
- U1 pad 40: /COL15 -> /ROW7
- U1 pad 41: /ROW1 -> /ROW6
Routing:
- net /COL13: track 539.6 -> 0.00 mm
- net Net-(D2:1-Pad1): track 501.8 -> 0.00 mm
- net /COL14: track 494.1 -> 0.00 mm
- net /COL11: track 752.1 -> 263.2 mm
- net /COL12: track 632.4 -> 187.7 mm
- net /ROW1: track 621.6 -> 228.1 mm
- net Net-(D3:1-Pad1): track 386.3 -> 0.00 mm
- net /COL15: track 334.5 -> 0.00 mm
- net GND: track 586.0 -> 897.0 mm
- net /ROW8: track 0.00 -> 302.0 mm
- net /ROW7: track 0.00 -> 291.3 mm
- net /ROW6: track 0.00 -> 280.1 mm
- net Net-("3"1-Pad1): track 257.6 -> 0.00 mm
- net VCC: track 302.3 -> 557.7 mm
- net Net-(D4:1-Pad1): track 231.6 -> 0.00 mm
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Other:
- board size 285.8 x 100.6 mm -> 285.8 x 98.5 mm

Commit message: enlarge trace width
Parts:
- moved D10:9 5.39 mm to (233.3, 153.0)
- moved D2:3 5.29 mm to (105.1, 99.0)
- moved D2:5 4.69 mm to (143.3, 99.0)
- moved D9:7 4.52 mm to (239.5, 150.8)
- moved R4 3.47 mm to (72.1, 147.8)
- moved R3 3.29 mm to (70.3, 147.8)
- moved D2:4 3.26 mm to (124.7, 99.0)
- moved D9:8 2.84 mm to (242.1, 150.8)
- moved D3:3 2.66 mm to (103.3, 100.0)
- moved D3:5 2.56 mm to (141.3, 100.0)
- moved D10:10 2.34 mm to (245.7, 155.0)
- moved D3:6 2.06 mm to (161.3, 100.0)
- moved D3:4 1.49 mm to (122.7, 100.0)
- moved D9:11 1.33 mm to (278.5, 164.0)
- moved D6:9 1.27 mm to (292.5, 97.6)
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Connections:
- net Net-(R3-Pad1) renamed /D-
- net Net-(R4-Pad1) renamed /D+
Routing:
- net /COL11: track 263.2 -> 214.0 mm
- net /ROW2: track 258.8 -> 233.5 mm
- net VCC: track 557.7 -> 578.4 mm
- net /D-: track 198.2 -> 218.7 mm
- net /D+: track 194.7 -> 212.7 mm
- net Net-(R1-Pad1): track 26.6 -> 39.1 mm
- net /ROW6: track 280.1 -> 292.3 mm
- net /ROW8: track 302.0 -> 314.2 mm
- net /ROW9: track 100.4 -> 88.5 mm
- net /ROW7: track 291.3 -> 302.9 mm
- net /COL10: track 212.8 -> 221.6 mm
- net /COL7: track 160.7 -> 169.1 mm
- net /COL9: track 152.5 -> 144.3 mm
- net GND: track 897.0 -> 905.0 mm
- net /COL5: track 186.3 -> 194.2 mm
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Other:
- board size 285.8 x 98.5 mm -> 285.8 x 97.7 mm
- net class Default: trace_width 0.25 -> 0.4

Commit message: redraw outline
Parts:
- moved R4 20.2 mm to (72.5, 127.7)
- moved R3 19.5 mm to (70.9, 128.3)
Routing:
- net /D+: track 212.7 -> 236.3 mm
- net Net-(J1-Pad3): track 299.1 -> 278.0 mm
- net Net-(J1-Pad2): track 299.0 -> 278.3 mm
- net /D-: track 218.7 -> 236.0 mm
- net GND: track 905.0 -> 900.8 mm
- net VCC: track 578.4 -> 576.0 mm
- net /ROW1: track 222.3 -> 223.9 mm
- net /ROW3: track 236.5 -> 238.0 mm
- net /ROW2: track 233.5 -> 235.0 mm

Commit message: fix left super size
Parts:
- L_CMD1: footprint TheKeebrary:MX_Plate_100H -> TheKeebrary:MX_Plate_150H
- moved D2:1 89.3 mm to (31.4, 34.5), turned to 270 degrees
- moved D10:9 86.3 mm to (179.9, 85.3)
- moved D3:1 85.6 mm to (42.0, 35.6), turned to 270 degrees
- moved D5:2 84.1 mm to (67.6, 114.2), turned to 90 degrees
- moved ALT1 83.0 mm to (63.1, 112.8)
- moved D9:9 80.6 mm to (228.2, 98.5)
- moved L_CMD1 80.0 mm to (86.9, 112.8)
- moved D9:7 79.9 mm to (194.2, 85.0)
- moved D9:10 79.8 mm to (231.6, 98.5)
- moved D5:4 79.6 mm to (149.8, 114.2), turned to 90 degrees
- moved D9:11 79.5 mm to (236.2, 96.8)
- moved D9:12 78.8 mm to (236.2, 100.0)
- moved D1:1 78.4 mm to (38.4, 33.6)
- moved D5:1 78.4 mm to (70.6, 114.2)
- moved D4:1 78.2 mm to (73.8, 113.1)
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Routing:
- net /ROW4: track 163.2 -> 120.9 mm
- net /COL2: track 234.2 -> 275.6 mm
- net Net-("K"1-Pad2): track 14.7 -> 53.3 mm
- net /COL4: track 150.0 -> 185.1 mm
- net /COL3: track 239.4 -> 268.6 mm
- net /COL9: track 144.3 -> 171.9 mm
- net Net-(CTRL1-Pad2): track 23.9 -> 50.3 mm
- net Net-("G"1-Pad2): track 16.8 -> 40.2 mm
- net Net-("U"1-Pad2): track 76.0 -> 55.1 mm
- net Net-("Y"1-Pad2): track 42.3 -> 62.4 mm
- net Net-(D2:1-Pad2): track 6.29 -> 20.3 mm
- net /ROW3: track 238.0 -> 226.4 mm
- net /COL10: track 221.6 -> 210.4 mm
- net Net-("X"1-Pad2): track 16.7 -> 26.1 mm
- net Net-("M"1-Pad2): track 2.88 -> 12.0 mm
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Other:
- board size 285.8 x 97.7 mm -> 285.8 x 98.6 mm

Commit message: optimize some path
Parts:
- moved R3 182.7 mm to (202.7, 118.0), turned to 270 degrees
- moved R4 179.2 mm to (200.9, 118.0), turned to 270 degrees
- moved D4:2 14.3 mm to (92.7, 113.0)
- moved D10:12 12.4 mm to (200.9, 93.7), turned to 90 degrees
- moved D10:8 8.62 mm to (179.9, 85.2)
- moved D10:7 8.54 mm to (179.9, 83.4)
- moved D10:11 8.11 mm to (202.9, 93.7), turned to 90 degrees
- moved D5:3 7.33 mm to (83.1, 114.0)
- moved D:7:7 6.01 mm to (190.9, 34.2)
- moved D9:8 5.53 mm to (218.9, 98.4)
- moved D7:10 4.81 mm to (252.9, 34.2)
- moved D10:9 4.40 mm to (184.3, 85.0)
- moved D10:10 4.27 mm to (204.9, 93.7)
- moved D7:9 4.21 mm to (235.3, 34.2)
- moved D5:6 2.94 mm to (161.3, 114.0)
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Routing:
- net Net-(J1-Pad2): track 278.9 -> 513.8 mm
- net Net-(J1-Pad3): track 278.9 -> 510.1 mm
- net /D-: track 232.2 -> 7.02 mm
- net /D+: track 230.4 -> 6.37 mm
- net /ROW10: track 70.2 -> 36.3 mm
- net /COL8: track 158.7 -> 128.3 mm
- net /COL3: track 268.6 -> 295.8 mm
- net Net-(D10:12-Pad2): track 44.9 -> 70.6 mm
- net /COL9: track 171.9 -> 149.2 mm
- net Net-(D10:11-Pad2): track 24.8 -> 47.0 mm
- net /COL7: track 175.2 -> 153.4 mm
- net GND: track 896.1 -> 914.0 mm
- net VCC: track 574.9 -> 588.4 mm
- net Net-("L"1-Pad2): track 40.4 -> 52.6 mm
- net /ROW7: track 303.3 -> 313.8 mm
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